File: hardware/tile/tile/coil_center.kicad_sch (KiCad schematic)
At the start: 6 parts, among them Q2 AO3400A

Commit message: added coils will improve them later
Parts:
- L1: renamed from L2; footprint footprints:coil_done -> (none)
- renumbered D7 to D6, Q2 to Q1, R14 to R11, R15 to R12, R16 to R13
Changed lines of the file:
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@@
 		(dnp no)
 		(fields_autoplaced yes)
-		(property "Reference" "R16"
+		(property "Reference" "R13"
 			(at 146.05 82.5499 0)
 			(effects
@@
 		(dnp no)
 		(fields_autoplaced yes)
-		(property "Reference" "D7"
+		(property "Reference" "D6"
 			(at 132.08 66.0399 90)
 			(effects
@@
 		(dnp no)
 		(fields_autoplaced yes)
-		(property "Reference" "#PWR026"
+		(property "Reference" "#PWR024"
 			(at 143.51 111.76 0)
 			(effects
@@
 		(dnp no)
 		(fields_autoplaced yes)
-		(property "Reference" "R15"
+		(property "Reference" "R12"
 			(at 135.89 97.7899 0)
 			(effects
@@
 		(dnp no)
 		(fields_autoplaced yes)
-		(property "Reference" "Q2"
+		(property "Reference" "Q1"
 			(at 147.32 93.9799 0)
 			(effects
@@
 		(dnp no)
 		(fields_autoplaced yes)
-		(property "Reference" "R14"
+		(property "Reference" "R11"
 			(at 127 88.9 90)
 			(effects
@@
 		(dnp no)
 		(fields_autoplaced yes)
-		(property "Reference" "L2"
+		(property "Reference" "L1"
 			(at 144.78 66.0399 0)
 			(effects
@@
 			)
 		)
-		(property "Footprint" "footprints:coil_done"
+		(property "Footprint" ""
 			(at 143.51 67.31 0)
 			(effects
@@
 		(dnp no)
 		(fields_autoplaced yes)
-		(property "Reference" "#PWR025"
+		(property "Reference" "#PWR023"
 			(at 143.51 57.15 0)
 			(effects
