File: hardware/tile/tile/connectors.kicad_sch (KiCad schematic)
At the start: 8 parts, among them J1 Conn_02x02_Counter_Clockwise, J2 Conn_02x02_Counter_Clockwise, J3 Conn_02x02_Counter_Clockwise, J4 Conn_02x02_Counter_Clockwise, J5 Conn_02x02_Counter_Clockwise, J6 Conn_02x02_Counter_Clockwise, J7 Conn_02x02_Counter_Clockwise, J8 Conn_02x02_Counter_Clockwise

Commit message: added coils will improve them later
Parts:
- J1, J2, J6: footprint (none) -> Connector_PinHeader_1.27mm:PinHeader_2x02_P1.27mm_Horizontal
- J3: renamed from J7; footprint (none) -> Connector_PinHeader_1.27mm:PinHeader_2x02_P1.27mm_Horizontal
- J4: renamed from J5; footprint (none) -> Connector_PinHeader_1.27mm:PinHeader_2x02_P1.27mm_Horizontal
- J5: renamed from J8; footprint (none) -> Connector_PinHeader_1.27mm:PinHeader_2x02_P1.27mm_Horizontal
- J7: renamed from J3; footprint (none) -> Connector_PinHeader_1.27mm:PinHeader_2x02_P1.27mm_Horizontal
- J8: renamed from J4; footprint (none) -> Connector_PinHeader_1.27mm:PinHeader_2x02_P1.27mm_Horizontal
Changed lines of the file:
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@@
 		(dnp no)
 		(fields_autoplaced yes)
-		(property "Reference" "#PWR037"
+		(property "Reference" "#PWR045"
 			(at 165.1 78.74 0)
 			(effects
@@
 			(project ""
 				(path "/0d1a434e-f7db-4824-ad3a-5d1d7a542c63/ff60e42f-16d6-4c76-b7db-3dc191d02d17"
-					(reference "#PWR037")
+					(reference "#PWR045")
 					(unit 1)
 				)
@@
 		(dnp no)
 		(fields_autoplaced yes)
-		(property "Reference" "#PWR034"
+		(property "Reference" "#PWR038"
 			(at 115.57 129.54 0)
 			(effects
@@
 			(project ""
 				(path "/0d1a434e-f7db-4824-ad3a-5d1d7a542c63/ff60e42f-16d6-4c76-b7db-3dc191d02d17"
-					(reference "#PWR034")
+					(reference "#PWR038")
 					(unit 1)
 				)
@@
 		(dnp no)
 		(fields_autoplaced yes)
-		(property "Reference" "#PWR028"
+		(property "Reference" "#PWR047"
 			(at 175.26 104.14 0)
 			(effects
@@
 			(project ""
 				(path "/0d1a434e-f7db-4824-ad3a-5d1d7a542c63/ff60e42f-16d6-4c76-b7db-3dc191d02d17"
-					(reference "#PWR028")
+					(reference "#PWR047")
 					(unit 1)
 				)
@@
 		(dnp no)
 		(fields_autoplaced yes)
-		(property "Reference" "#PWR022"
+		(property "Reference" "#PWR035"
 			(at 82.55 104.14 0)
 			(effects
@@
 			(project ""
 				(path "/0d1a434e-f7db-4824-ad3a-5d1d7a542c63/ff60e42f-16d6-4c76-b7db-3dc191d02d17"
-					(reference "#PWR022")
+					(reference "#PWR035")
 					(unit 1)
 				)
@@
 		(dnp no)
 		(fields_autoplaced yes)
-		(property "Reference" "#PWR036"
+		(property "Reference" "#PWR048"
 			(at 165.1 106.68 0)
 			(effects
@@
 			(project ""
 				(path "/0d1a434e-f7db-4824-ad3a-5d1d7a542c63/ff60e42f-16d6-4c76-b7db-3dc191d02d17"
-					(reference "#PWR036")
+					(reference "#PWR048")
 					(unit 1)
 				)
@@
 		(dnp no)
 		(fields_autoplaced yes)
-		(property "Reference" "#PWR033"
+		(property "Reference" "#PWR036"
 			(at 92.71 106.68 0)
 			(effects
@@
 			(project ""
 				(path "/0d1a434e-f7db-4824-ad3a-5d1d7a542c63/ff60e42f-16d6-4c76-b7db-3dc191d02d17"
-					(reference "#PWR033")
+					(reference "#PWR036")
 					(unit 1)
 				)
@@
 			)
 		)
-		(property "Footprint" ""
+		(property "Footprint" "Connector_PinHeader_1.27mm:PinHeader_2x02_P1.27mm_Horizontal"
 			(at 93.98 78.74 0)
 			(effects
@@
 		(dnp no)
 		(fields_autoplaced yes)
-		(property "Reference" "#PWR032"
+		(property "Reference" "#PWR033"
 			(at 92.71 78.74 0)
 			(effects
@@
 			(project ""
 				(path "/0d1a434e-f7db-4824-ad3a-5d1d7a542c63/ff60e42f-16d6-4c76-b7db-3dc191d02d17"
-					(reference "#PWR032")
+					(reference "#PWR033")
 					(unit 1)
 				)
@@
 		(dnp no)
 		(fields_autoplaced yes)
-		(property "Reference" "J4"
+		(property "Reference" "J8"
 			(at 162.56 97.79 0)
 			(effects
@@
 			)
 		)
-		(property "Footprint" ""
+		(property "Footprint" "Connector_PinHeader_1.27mm:PinHeader_2x02_P1.27mm_Horizontal"
 			(at 161.29 104.14 0)
 			(effects
@@
 			(project "tile"
 				(path "/0d1a434e-f7db-4824-ad3a-5d1d7a542c63/ff60e42f-16d6-4c76-b7db-3dc191d02d17"
-					(reference "J4")
+					(reference "J8")
 					(unit 1)
 				)
@@
 		(dnp no)
 		(fields_autoplaced yes)
-		(property "Reference" "#PWR029"
+		(property "Reference" "#PWR046"
 			(at 175.26 81.28 0)
 			(effects
@@
 			(project ""
 				(path "/0d1a434e-f7db-4824-ad3a-5d1d7a542c63/ff60e42f-16d6-4c76-b7db-3dc191d02d17"
-					(reference "#PWR029")
+					(reference "#PWR046")
 					(unit 1)
 				)
@@
 		(dnp no)
 		(fields_autoplaced yes)
-		(property "Reference" "#PWR038"
+		(property "Reference" "#PWR043"
 			(at 143.51 57.15 0)
 			(effects
@@
 			(project ""
 				(path "/0d1a434e-f7db-4824-ad3a-5d1d7a542c63/ff60e42f-16d6-4c76-b7db-3dc191d02d17"
-					(reference "#PWR038")
+					(reference "#PWR043")
 					(unit 1)
 				)
@@
 		(dnp no)
 		(fields_autoplaced yes)
-		(property "Reference" "#PWR035"
+		(property "Reference" "#PWR044"
 			(at 143.51 129.54 0)
 			(effects
@@
 			(project ""
 				(path "/0d1a434e-f7db-4824-ad3a-5d1d7a542c63/ff60e42f-16d6-4c76-b7db-3dc191d02d17"
-					(reference "#PWR035")
+					(reference "#PWR044")
 					(unit 1)
 				)
@@
 		(dnp no)
 		(fields_autoplaced yes)
-		(property "Reference" "#PWR039"
+		(property "Reference" "#PWR037"
 			(at 115.57 57.15 0)
 			(effects
@@
 			(project ""
 				(path "/0d1a434e-f7db-4824-ad3a-5d1d7a542c63/ff60e42f-16d6-4c76-b7db-3dc191d02d17"
-					(reference "#PWR039")
+					(reference "#PWR037")
 					(unit 1)
 				)
@@
 		(dnp no)
 		(fields_autoplaced yes)
-		(property "Reference" "#PWR024"
+		(property "Reference" "#PWR040"
 			(at 118.11 139.7 0)
 			(effects
@@
 			(project ""
 				(path "/0d1a434e-f7db-4824-ad3a-5d1d7a542c63/ff60e42f-16d6-4c76-b7db-3dc191d02d17"
-					(reference "#PWR024")
+					(reference "#PWR040")
 					(unit 1)
 				)
@@
 		(dnp no)
 		(fields_autoplaced yes)
-		(property "Reference" "J7"
+		(property "Reference" "J3"
 			(at 109.22 59.69 0)
 			(effects
@@
 			)
 		)
-		(property "Footprint" ""
+		(property "Footprint" "Connector_PinHeader_1.27mm:PinHeader_2x02_P1.27mm_Horizontal"
 			(at 115.57 60.96 0)
 			(effects
@@
 			(project "tile"
 				(path "/0d1a434e-f7db-4824-ad3a-5d1d7a542c63/ff60e42f-16d6-4c76-b7db-3dc191d02d17"
-					(reference "J7")
+					(reference "J3")
 					(unit 1)
 				)
@@
 		(dnp no)
 		(fields_autoplaced yes)
-		(property "Reference" "#PWR026"
+		(property "Reference" "#PWR042"
 			(at 140.97 139.7 0)
 			(effects
@@
 			(project ""
 				(path "/0d1a434e-f7db-4824-ad3a-5d1d7a542c63/ff60e42f-16d6-4c76-b7db-3dc191d02d17"
-					(reference "#PWR026")
+					(reference "#PWR042")
 					(unit 1)
 				)
@@
 		(dnp no)
 		(fields_autoplaced yes)
-		(property "Reference" "J8"
+		(property "Reference" "J5"
 			(at 134.62 59.69 0)
 			(effects
@@
 			)
 		)
-		(property "Footprint" ""
+		(property "Footprint" "Connector_PinHeader_1.27mm:PinHeader_2x02_P1.27mm_Horizontal"
 			(at 140.97 60.96 0)
 			(effects
@@
 			(project "tile"
 				(path "/0d1a434e-f7db-4824-ad3a-5d1d7a542c63/ff60e42f-16d6-4c76-b7db-3dc191d02d17"
-					(reference "J8")
+					(reference "J5")
 					(unit 1)
 				)
@@
 		(dnp no)
 		(fields_autoplaced yes)
-		(property "Reference" "J3"
+		(property "Reference" "J7"
 			(at 162.56 72.39 0)
 			(effects
@@
 			)
 		)
-		(property "Footprint" ""
+		(property "Footprint" "Connector_PinHeader_1.27mm:PinHeader_2x02_P1.27mm_Horizontal"
 			(at 161.29 78.74 0)
 			(effects
@@
 			(project "tile"
 				(path "/0d1a434e-f7db-4824-ad3a-5d1d7a542c63/ff60e42f-16d6-4c76-b7db-3dc191d02d17"
-					(reference "J3")
+					(reference "J7")
 					(unit 1)
 				)
@@
 		(dnp no)
 		(fields_autoplaced yes)
-		(property "Reference" "#PWR030"
+		(property "Reference" "#PWR041"
 			(at 140.97 46.99 0)
 			(effects
@@
 			(project ""
 				(path "/0d1a434e-f7db-4824-ad3a-5d1d7a542c63/ff60e42f-16d6-4c76-b7db-3dc191d02d17"
-					(reference "#PWR030")
+					(reference "#PWR041")
 					(unit 1)
 				)
@@
 		(dnp no)
 		(fields_autoplaced yes)
-		(property "Reference" "#PWR031"
+		(property "Reference" "#PWR039"
 			(at 118.11 46.99 0)
 			(effects
@@
 			(project ""
 				(path "/0d1a434e-f7db-4824-ad3a-5d1d7a542c63/ff60e42f-16d6-4c76-b7db-3dc191d02d17"
-					(reference "#PWR031")
+					(reference "#PWR039")
 					(unit 1)
 				)
@@
 			)
 		)
-		(property "Footprint" ""
+		(property "Footprint" "Connector_PinHeader_1.27mm:PinHeader_2x02_P1.27mm_Horizontal"
 			(at 93.98 104.14 0)
 			(effects
@@
 			)
 		)
-		(property "Footprint" ""
+		(property "Footprint" "Connector_PinHeader_1.27mm:PinHeader_2x02_P1.27mm_Horizontal"
 			(at 140.97 128.27 0)
 			(effects
@@
 		(dnp no)
 		(fields_autoplaced yes)
-		(property "Reference" "#PWR020"
+		(property "Reference" "#PWR034"
 			(at 82.55 81.28 0)
 			(effects
@@
 			(project ""
 				(path "/0d1a434e-f7db-4824-ad3a-5d1d7a542c63/ff60e42f-16d6-4c76-b7db-3dc191d02d17"
-					(reference "#PWR020")
+					(reference "#PWR034")
 					(unit 1)
 				)
@@
 		(dnp no)
 		(fields_autoplaced yes)
-		(property "Reference" "J5"
+		(property "Reference" "J4"
 			(at 109.22 127 0)
 			(effects
@@
 			)
 		)
-		(property "Footprint" ""
+		(property "Footprint" "Connector_PinHeader_1.27mm:PinHeader_2x02_P1.27mm_Horizontal"
 			(at 115.57 128.27 0)
 			(effects
@@
 			(project "tile"
 				(path "/0d1a434e-f7db-4824-ad3a-5d1d7a542c63/ff60e42f-16d6-4c76-b7db-3dc191d02d17"
-					(reference "J5")
-					(unit 1)
-				)
+					(reference "J4")
+					(unit 1)
+				)
